Commit message: Updated PID files

File: description/urdf/imu.xacro (robot description, xacro)
@@ -1,33 +1,104 @@
 <?xml version="1.0"?>
 <robot xmlns:xacro="http://www.ros.org/wiki/xacro" >
-    <joint name="imu_joint" type="fixed">
-        <parent link="chassis"/>
-        <child link="imu_link"/>
-        <origin xyz="-0.05 0 0.55" rpy="0 0 0"/>
-    </joint>
-    <link name="imu_link">
-    </link>
-  <gazebo reference="imu_link">
-    <gravity>true</gravity>
-    <sensor name="imu_sensor" type="imu">
-      <always_on>true</always_on>
-      <update_rate>100</update_rate>
-      <visualize>true</visualize>
-      <topic>__default_topic__</topic>
-      <plugin filename="libgazebo_ros_imu_sensor.so" name="imu_plugin">
-        <ros>
-            <remapping>~/out:=/imu</remapping>
-        </ros>
-        <topicName>imu</topicName>
-        <bodyName>imu_link</bodyName>
-        <updateRateHZ>10.0</updateRateHZ>
-        <gaussianNoise>0.0</gaussianNoise>
-        <xyzOffset>0 0 0</xyzOffset>
-        <rpyOffset>0 0 0</rpyOffset>
-        <frameName>imu_link</frameName>
-        <initialOrientationAsReference>false</initialOrientationAsReference>
-      </plugin>
-      <pose>0 0 0 0 0 0</pose>
-    </sensor>
-  </gazebo>
+  <joint name="imu_joint" type="fixed">
+    <parent link="chassis" />
+    <child link="imu" />
+    <origin xyz="0 0 0.145" rpy="0 0 0" />
+  </joint>
+  <link name="imu">
+    <visual>
+      <origin xyz="0 0 0" rpy="0 0 0" />
+      <geometry>
+        <box size="0.01 0.01 0.01" />
+      </geometry>
+      <material name="red"/>
+    </visual>
+    <collision>
+      <origin xyz="0 0 0" rpy="0 0 0" />
+      <geometry>
+        <box size="0.01 0.01 0.01" />
+      </geometry>
+    </collision>
+    <inertial>
+      <origin xyz="0 0 0" rpy="0 0 0" />
+      <mass value="1" />
+      <inertia ixx="0.000016666666666666667" ixy="0" ixz="0" iyy="0.000016666666666666667" iyz="0" izz="0.000016666666666666667" />
+    </inertial>
+  </link>
+ <gazebo reference="imu">
+   <sensor name="mpu6050_imu" type="imu">
+    <plugin name="imu_controller" filename="libgazebo_ros_imu_sensor.so">
+      <frame_name>imu</frame_name>
+       <ros>
+         <remapping>~/out:=/imu</remapping>
+       </ros>
+      <initial_orientation_as_reference>false</initial_orientation_as_reference>
+    </plugin>
+     <always_on>true</always_on>
+     <update_rate>100</update_rate>
+     <visualize>true</visualize>
+     <imu>
+       <angular_velocity>
+         <x>
+           <noise type="gaussian">
+             <mean>0.0</mean>
+             <stddev>2e-4</stddev>
+           </noise>
+         </x>
+         <y>
+           <noise type="gaussian">
+             <mean>0.0</mean>
+             <stddev>2e-4</stddev>
+           </noise>
+         </y>
+         <z>
+           <noise type="gaussian">
+             <mean>0.0</mean>
+             <stddev>2e-4</stddev>
+           </noise>
+         </z>
+       </angular_velocity>
+       <linear_acceleration>
+         <x>
+           <noise type="gaussian">
+             <mean>0.0</mean>
+             <stddev>1.7e-2</stddev>
+           </noise>
+         </x>
+         <y>
+           <noise type="gaussian">
+             <mean>0.0</mean>
+             <stddev>1.7e-2</stddev>
+           </noise>
+         </y>
+         <z>
+           <noise type="gaussian">
+             <mean>0.0</mean>
+             <stddev>1.7e-2</stddev>
+           </noise>
+         </z>
+       </linear_acceleration>
+       <orientation>
+         <x>
+           <noise type="gaussian">
+              <mean>0.0</mean>
+              <stddev>2e-3</stddev>
+            </noise>
+          </x>
+          <y>
+            <noise type="gaussian">
+              <mean>0.0</mean>
+              <stddev>2e-3</stddev>
+            </noise>
+          </y>
+          <z>
+            <noise type="gaussian">
+              <mean>0.0</mean>
+              <stddev>2e-3</stddev>
+            </noise>
+          </z>
+        </orientation>
+     </imu>
+   </sensor>
+ </gazebo>
 </robot>

File: description/urdf/lidar.xacro (robot description, xacro)
@@ -1,26 +1,30 @@
 <?xml version="1.0"?>
 <robot xmlns:xacro="http://www.ros.org/wiki/xacro" >
-    <joint name="laser_joint" type="fixed">
-        <parent link="chassis"/>
-        <child link="laser_frame"/>
-        <origin xyz="0.05 0 0.25" rpy="0 0 0"/>
-    </joint>
-    <link name="laser_frame">
+    <link name="laser">
         <visual>
-            <geometry>
-                <cylinder radius="0.05" length="0.04"/>
-            </geometry>
-            <material name="black"/>
+        <origin xyz="0 0 0" rpy="0 0 0" />
+        <geometry>
+            <cylinder radius="0.03000000000000003" length="0.04" />
+        </geometry>
+        <material name="black"/>
         </visual>
         <collision>
-            <geometry>
-                <cylinder radius="0.05" length="0.04"/>
-            </geometry>
+        <origin xyz="0 0 0" rpy="0 0 0" />
+        <geometry>
+            <cylinder radius="0.03000000000000003" length="0.04" />
+        </geometry>
         </collision>
-        <xacro:inertial_cylinder mass="0.1" length="0.04" radius="0.05">
-            <origin xyz="0 0 0" rpy="0 0 0"/>
-        </xacro:inertial_cylinder>
+        <inertial>
+        <origin xyz="0 0 0" rpy="0 0 0" />
+        <mass value="0.11" />
+        <inertia ixx="0.00013199999999999996" ixy="0" ixz="0" iyy="0.00019799999999999996" iyz="0" izz="0.00013199999999999996" />
+        </inertial>
     </link>
-    <gazebo reference="laser_frame">
+    <joint name="laser_joint" type="fixed">
+        <parent link="base_link" />
+        <child link="laser" />
+        <origin xyz="0.04 0 0.155" rpy="0 0 0" />
+    </joint>
+    <gazebo reference="laser">
         <material>Gazebo/Black</material>
         <sensor name="laser" type="ray">
@@ -38,5 +42,5 @@
                 <range>
                     <min>0.3</min>
-                    <max>20</max>
+                    <max>12</max>
                 </range>
             </ray>
@@ -46,5 +50,5 @@
                 </ros>
                 <output_type>sensor_msgs/LaserScan</output_type>
-                <frame_name>laser_frame</frame_name>
+                <frame_name>laser</frame_name>
             </plugin>
         </sensor>

File: description/urdf/robot.urdf.xacro (robot description, xacro)
@@ -1,7 +1,7 @@
 <?xml version="1.0"?>
 <robot xmlns:xacro="http://www.ros.org/wiki/xacro"  name="robot">
-    <xacro:arg name="sim_mode" default="false"/>
+    <xacro:arg name="sim_mode" default="false"/> -->
+    <xacro:include filename="ros2_control.xacro" />
     <xacro:include filename="robot_core.xacro" />
-    <xacro:include filename="ros2_control.xacro" />
     <xacro:include filename="lidar.xacro" />
     <xacro:include filename="imu.xacro" />

File: description/urdf/robot_core.xacro (robot description, xacro)
@@ -1,21 +1,3 @@
-<?xml version="1.0"?>
-<robot xmlns:xacro="http://www.ros.org/wiki/xacro" >
-    <xacro:include filename="inertial_macros.xacro"/>
-    <xacro:property name="chassis_width" value="0.6"/>        <!-- Length of the chassis in meters -->
-    <xacro:property name="chassis_length" value="0.2"/>        <!-- Width of the chassis in meters -->
-    <xacro:property name="chassis_height" value="0.2"/>       <!-- Height of the chassis in meters -->
-    <xacro:property name="chassis_mass" value="5.0"/>         <!-- Mass of the chassis in kilograms -->
-    <xacro:property name="wheel_radius" value="0.1651"/>       <!-- Radius of the wheel in meters (6.5 inches) -->
-    <xacro:property name="wheel_thickness" value="0.0635"/>    <!-- Thickness of the wheel in meters (2.5 inches) -->
-    <xacro:property name="wheel_mass" value="1.3"/>            <!-- Mass of the wheel in kilograms (2.9 lbs) -->
-    <xacro:property name="wheel_offset_x" value="0.0"/>        <!-- Offset of the wheel along the x-axis in meters -->
-    <xacro:property name="wheel_offset_y" value="0.331"/>       <!-- Offset of the wheel along the y-axis in meters -->
-    <xacro:property name="wheel_offset_z" value="0.01"/>       <!-- Offset of the wheel along the z-axis in meters -->
-    <xacro:property name="rod_length" value="0.5"/>       <!-- Offset of the wheel along the z-axis in meters -->
-    <xacro:property name="rod_thickness" value="0.02"/>       <!-- Offset of the wheel along the z-axis in meters -->
-    <xacro:property name="rod_mass" value="0.2"/>       <!-- Offset of the wheel along the z-axis in meters -->
-    <xacro:property name="rod_offset_x" value="-0.05"/>       <!-- Offset of the wheel along the z-axis in meters -->
-    <xacro:property name="rod_offset_y" value="0.0"/>       <!-- Offset of the wheel along the z-axis in meters -->
-    <xacro:property name="rod_offset_z" value="0.25"/>       <!-- Offset of the wheel along the z-axis in meters -->
+<robot name="GeneratedRobot">
     <material name="white">
         <color rgba="1 1 1 1" />
@@ -33,117 +15,115 @@
         <color rgba="1 0 0 1"/>
     </material>
-        <!-- BASE LINK -->
-    <link name="base_link">
+    <link name = "base_link">
+        <origin xyz="0.0 0.0 0.08" rpy="0.0 0.0 0.0"/>
     </link>
-    <!-- BASE_FOOTPRINT LINK -->
-    <joint name="base_footprint_joint" type="fixed">
-        <parent link="base_link"/>
-        <child link="base_footprint"/>
-        <origin xyz="0 0 0" rpy="0 0 0"/>
-    </joint>
-    <link name="base_footprint">
-    </link>
-        <!-- CHASSIS LINK -->
     <joint name="chassis_joint" type="fixed">
+        <origin xyz="0.0 0.0 0.0" rpy="0.0 0.0 0.0"/>
         <parent link="base_link"/>
         <child link="chassis"/>
-        <origin xyz="0 0 ${-wheel_offset_z}"/>
     </joint>
+    <!-- CHASSIS LINK -->
     <link name="chassis">
         <visual>
-            <origin xyz="0 0 ${chassis_height/2}"/>
+            <origin xyz="0 0 0.05" rpy="0 0 0" />
             <geometry>
-                <box size="${chassis_length} ${chassis_width} ${chassis_height}"/>
+                <box size="0.15 0.3 0.12" />
             </geometry>
             <material name="orange"/>
         </visual>
+        <visual>
+            <origin xyz="0.0 0.0 0.1" rpy="0.0 0.0 0.0"/>
+            <geometry>
+                <box size="0.25 0.3 0.08"/>
+            </geometry>
+            <material name = "orange"/>
+        </visual>
         <collision>
-            <origin xyz="0 0 ${chassis_height/2}"/>
+            <origin xyz="0 0 0.08" rpy="0 0 0" />
             <geometry>
-                <box size="${chassis_length} ${chassis_width} ${chassis_height}"/>
+                <box size="0.18 0.3 0.15" />
             </geometry>
         </collision>
-        <xacro:inertial_box mass="${chassis_mass}" x="${chassis_length}" y="${chassis_width}" z="${chassis_height}">
-            <origin xyz="${chassis_length/2} 0 ${chassis_height/2}" rpy="0 0 0"/>
-        </xacro:inertial_box>
+        <collision>
+            <origin xyz="0.0 0.0 0.1" rpy="0.0 0.0 0.0"/>
+            <geometry>
+                <box size="0.25 0.3 0.08"/>
+            </geometry>
+            <material name = "orange"/>
+        </collision>
+        <inertial>
+            <origin xyz="0 0 0.08" rpy="0 0 0" />
+            <mass value="7"/>
+            <inertia ixx="0.061" ixy="0" ixz="0" iyy="0.022" iyz="0" izz="0.066" />
+        </inertial>
     </link>
     <gazebo reference="chassis">
         <material>Gazebo/Orange</material>
     </gazebo>
-    <!-- LEFT WHEEL LINK -->
-    <joint name="left_wheel_joint" type="continuous">
+    <joint name="base_footprint_joint" type="fixed">
         <parent link="base_link"/>
-        <child link="left_wheel"/>
-        <origin xyz="0 ${wheel_offset_y} 0" rpy="-${pi/2} 0 0" />
-        <axis xyz="0 0 1"/>
+        <child link="base_footprint"/>
+        <origin xyz="0.0 0.0 0.0" rpy="0.0 0.0 0.0"/>
     </joint>
+    <link name="base_footprint">
+    </link>
+    <!-- LEFT WHEEL -->
     <link name="left_wheel">
         <visual>
+            <origin xyz="0 0 0" rpy="0 0 0" />
             <geometry>
-                <cylinder radius="${wheel_radius}" length="${wheel_thickness}"/>
-            </geometry>
-            <material name="blue"/>
-        </visual>
-        <collision>
-            <geometry>
-                <sphere radius="${wheel_radius}"/>
-            </geometry>
-        </collision>
-        <xacro:inertial_cylinder mass="${wheel_mass}" length="${wheel_thickness}" radius="${wheel_radius}">
-            <origin xyz="0 0 0" rpy="0 0 0"/>
-        </xacro:inertial_cylinder>
-    </link>
-    <gazebo reference="left_wheel">
-        <material>Gazebo/Blue</material>
-    </gazebo>
-    <!-- RIGHT WHEEL LINK -->
-    <joint name="right_wheel_joint" type="continuous">
-        <parent link="base_link"/>
-        <child link="right_wheel"/>
-        <origin xyz="0 ${-wheel_offset_y} 0" rpy="${pi/2} 0 0" />
-        <axis xyz="0 0 -1"/>
-    </joint>
-    <link name="right_wheel">
-        <visual>
-            <geometry>
-                <cylinder radius="${wheel_radius}" length="${wheel_thickness}"/>
-            </geometry>
-            <material name="blue"/>
-        </visual>
-        <collision>
-            <geometry>
-                <sphere radius="${wheel_radius}"/>
-            </geometry>
-        </collision>
-        <xacro:inertial_cylinder mass="${wheel_mass}" length="${wheel_thickness}" radius="${wheel_radius}">
-            <origin xyz="0 0 0" rpy="0 0 0"/>
-        </xacro:inertial_cylinder>
-    </link>
-    <gazebo reference="right_wheel">
-        <material>Gazebo/Blue</material>
-    </gazebo>
-    <joint name="rod_joint" type="fixed">
-        <parent link="base_link"/>
-        <child link="rod_link"/>
-        <origin xyz="${rod_offset_x} ${rod_offset_y} ${rod_offset_z}"/>
-    </joint>
-    <link name="rod_link">
-        <visual>
-            <geometry>
-                <cylinder radius="${rod_thickness}" length="${rod_length}"/>
+                <cylinder radius="0.08499999999999996" length="0.0635" />
             </geometry>
             <material name="white"/>
         </visual>
         <collision>
+            <origin xyz="0 0 0" rpy="0 0 0" />
             <geometry>
-                <cylinder radius="${rod_thickness}" length="${rod_length}"/>
+                <cylinder radius="0.08499999999999996" length="0.0635" />
+            </geometry>
+        </collision>
+        <inertial>
+            <origin xyz="0 0 0" rpy="0 0 0" />
+            <mass value="2" />
+            <inertia ixx="0.019266666666666668" ixy="0" ixz="0" iyy="0.028900000000000006" iyz="0" izz="0.019266666666666668" />
+        </inertial>
+    </link>
+    <joint name="left_wheel_joint" type="continuous">
+        <parent link="chassis" />
+        <child link="left_wheel" />
+        <origin xyz="0 0.18 0" rpy="1.5707963267948963 0 0" />
+        <axis xyz="0 0 1"/>
+    </joint>
+    <gazebo reference="left_wheel">
+        <material>Gazebo/White</material>
+    </gazebo>
+    <!-- RIGHT WHEEL -->
+    <link name="right_wheel">
+        <visual>
+            <origin xyz="0 0 0" rpy="0 0 0" />
+            <geometry>
+                <cylinder radius="0.085" length="0.0635" />
             </geometry>
             <material name="white"/>
+        </visual>
+        <collision>
+            <origin xyz="0 0 0" rpy="0 0 0" />
+            <geometry>
+                <cylinder radius="0.085" length="0.0635" />
+            </geometry>
         </collision>
-        <xacro:inertial_cylinder mass="${rod_mass}" length="${rod_length}" radius="${rod_thickness}">
-            <origin xyz="0 0 0" rpy="0 0 0"/>
-        </xacro:inertial_cylinder>
+        <inertial>
+            <origin xyz="0 0 0" rpy="0 0 0" />
+            <mass value="1" />
+            <inertia ixx="0" ixy="0" ixz="0" iyy="0" iyz="0" izz="0" />
+        </inertial>
     </link>
-    <gazebo reference="rod_link">
+    <joint name="right_wheel_joint" type="continuous">
+        <parent link="chassis" />
+        <child link="right_wheel" />
+        <origin xyz="0 -0.18 0" rpy="1.5707963267948966 0 0.030840783524403125" />
+        <axis xyz="0 0 1"/>
+    </joint>
+    <gazebo reference="right_wheel">
         <material>Gazebo/White</material>
     </gazebo>

File: description/urdf/ros2_control.xacro (robot description, xacro)
@@ -7,6 +7,6 @@
         <joint name="left_wheel_joint">
             <command_interface name="velocity">
-                <param name="min">-10</param>
-                <param name="max">10</param>
+                <param name="min">-5</param>
+                <param name="max">5</param>
             </command_interface>
             <state_interface name="velocity"/>
@@ -15,6 +15,6 @@
         <joint name="right_wheel_joint">
             <command_interface name="velocity">
-                <param name="min">-10</param>
-                <param name="max">10</param>
+                <param name="min">-5</param>
+                <param name="max">5</param>
             </command_interface>
             <state_interface name="velocity"/>
